File: kablampad.kicad_pcb (KiCad board)
At the start: 2 copper layers, 107.2 x 66.7 mm, 29 parts, among them U1 RP2040_Zero

Commit message: made kablamboard v1, idk how i'm gonna merge later (but that's a future problem, yaknow?)
Parts:
- removed the REF** at (152.4, 116.7)
- removed the REF** at (54.8, 116.7)
- removed the REF** at (54.8, 54.8)
- removed the REF** at (152.4, 54.8)
- added D13: Diode, ScottoKeebs_Components:Diode_DO-35, F.Cu at (91.2, 70.5)
- added D14: Diode, ScottoKeebs_Components:Diode_DO-35, F.Cu at (107.5, 81.5)
- added D15: Diode, ScottoKeebs_Components:Diode_DO-35, F.Cu at (110.9, 88.8)
- added D16: Diode, ScottoKeebs_Components:Diode_DO-35, F.Cu at (189.3, 81.6)
- added D17: Diode, ScottoKeebs_Components:Diode_DO-35, F.Cu at (207.2, 75.0)
- added D18: Diode, ScottoKeebs_Components:Diode_DO-35, F.Cu at (223.5, 64.1)
- added D19: Diode, ScottoKeebs_Components:Diode_DO-35, F.Cu at (241.0, 56.6)
- added D20: Diode, ScottoKeebs_Components:Diode_DO-35, F.Cu at (251.9, 69.9)
- added D21: Diode, ScottoKeebs_Components:Diode_DO-35, F.Cu at (45.6, 84.3)
- added D22: Diode, ScottoKeebs_Components:Diode_DO-35, F.Cu at (66.0, 84.1)
- added D23: Diode, ScottoKeebs_Components:Diode_DO-35, F.Cu at (84.7, 88.4)
- added D24: Diode, ScottoKeebs_Components:Diode_DO-35, F.Cu at (100.9, 99.4)
- added D25: Diode, ScottoKeebs_Components:Diode_DO-35, F.Cu at (104.4, 106.7)
- added D26: Diode, ScottoKeebs_Components:Diode_DO-35, F.Cu at (195.8, 99.5)
- added D27: Diode, ScottoKeebs_Components:Diode_DO-35, F.Cu at (213.7, 92.9)
- added D28: Diode, ScottoKeebs_Components:Diode_DO-35, F.Cu at (230.0, 82.0)
- added D29: Diode, ScottoKeebs_Components:Diode_DO-35, F.Cu at (245.1, 67.8)
- added D30: Diode, ScottoKeebs_Components:Diode_DO-35, F.Cu at (249.5, 79.9)
- added D31: Diode, ScottoKeebs_Components:Diode_DO-35, F.Cu at (92.4, 104.9)
- added D32: Diode, ScottoKeebs_Components:Diode_DO-35, F.Cu at (105.7, 122.1)
- added D33: Diode, ScottoKeebs_Components:Diode_DO-35, F.Cu at (123.8, 135.2)
- added D34: Diode, ScottoKeebs_Components:Diode_DO-35, F.Cu at (172.9, 135.2)
- added D35: Diode, ScottoKeebs_Components:Diode_DO-35, F.Cu at (191.1, 122.2)
- added D36: Diode, ScottoKeebs_Components:Diode_DO-35, F.Cu at (195.0, 108.4)
- added D37: Diode, ScottoKeebs_Components:Diode_DO-35, F.Cu at (144.6, 119.7)
- added REF**: MountingHole_2.2mm_M2, MountingHole:MountingHole_2.2mm_M2, F.Cu at (21.3, 83.3)
- added REF**: MountingHole_2.2mm_M2, MountingHole:MountingHole_2.2mm_M2, F.Cu at (44.3, 21.3)
- added REF**: MountingHole_2.2mm_M2, MountingHole:MountingHole_2.2mm_M2, F.Cu at (274.3, 83.3)
- added REF**: MountingHole_2.2mm_M2, MountingHole:MountingHole_2.2mm_M2, F.Cu at (148.3, 154.3)
- added REF**: MountingHole_2.2mm_M2, MountingHole:MountingHole_2.2mm_M2, F.Cu at (250.8, 21.3)
- added REF**: MountingHole_2.2mm_M2, MountingHole:MountingHole_2.2mm_M2, F.Cu at (148.3, 56.3)
- added S13: Keyswitch, ScottoKeebs_Hotswap:Hotswap_MX_1.00u, F.Cu at (83.5, 63.6)
- added S14: Keyswitch, ScottoKeebs_Hotswap:Hotswap_MX_1.00u, F.Cu at (99.8, 74.6)
- added S15: Keyswitch, ScottoKeebs_Hotswap:Hotswap_MX_1.00u, F.Cu at (117.7, 81.1)
- added S16: Keyswitch, ScottoKeebs_Hotswap:Hotswap_MX_1.00u, F.Cu at (179.0, 81.2)
- added S17: Keyswitch, ScottoKeebs_Hotswap:Hotswap_MX_1.00u, F.Cu at (196.9, 74.7)
- added S18: Keyswitch, ScottoKeebs_Hotswap:Hotswap_MX_1.00u, F.Cu at (213.2, 63.7)
- added S19: Keyswitch, ScottoKeebs_Hotswap:Hotswap_MX_1.00u, F.Cu at (231.9, 59.5)
- added S20: Keyswitch, ScottoKeebs_Hotswap:Hotswap_MX_1.00u, F.Cu at (252.3, 59.7)
- added S21: Keyswitch, ScottoKeebs_Hotswap:Hotswap_MX_1.00u, F.Cu at (38.0, 77.5)
- added S22: Keyswitch, ScottoKeebs_Hotswap:Hotswap_MX_1.00u, F.Cu at (58.3, 77.3)
- added S23: Keyswitch, ScottoKeebs_Hotswap:Hotswap_MX_1.00u, F.Cu at (77.0, 81.5)
- added S24: Keyswitch, ScottoKeebs_Hotswap:Hotswap_MX_1.00u, F.Cu at (93.3, 92.5)
- added S25: Keyswitch, ScottoKeebs_Hotswap:Hotswap_MX_1.00u, F.Cu at (111.2, 99.0)
- added S26: Keyswitch, ScottoKeebs_Hotswap:Hotswap_MX_1.00u, F.Cu at (185.6, 99.1)
- added S27: Keyswitch, ScottoKeebs_Hotswap:Hotswap_MX_1.00u, F.Cu at (203.5, 92.6)
- added S28: Keyswitch, ScottoKeebs_Hotswap:Hotswap_MX_1.00u, F.Cu at (219.7, 81.6)
- added S29: Keyswitch, ScottoKeebs_Hotswap:Hotswap_MX_1.00u, F.Cu at (238.4, 77.4)
- added S30: Keyswitch, ScottoKeebs_Hotswap:Hotswap_MX_1.00u, F.Cu at (258.8, 77.6)
- added S31: Keyswitch, ScottoKeebs_Hotswap:Hotswap_MX_1.00u, F.Cu at (94.9, 115.9)
- added S32: Keyswitch, ScottoKeebs_Hotswap:Hotswap_MX_1.00u, F.Cu at (114.6, 125.7)
- added S33: Keyswitch, ScottoKeebs_Hotswap:Hotswap_MX_1.00u, F.Cu at (131.0, 141.6)
- added S34: Keyswitch, ScottoKeebs_Hotswap:Hotswap_MX_1.00u, F.Cu at (165.6, 141.6)
- added S35: Keyswitch, ScottoKeebs_Hotswap:Hotswap_MX_1.00u, F.Cu at (182.1, 125.8)
- added S36: Keyswitch, ScottoKeebs_Hotswap:Hotswap_MX_1.00u, F.Cu at (201.8, 116.0)
- added SW1: RotaryEncoder_Switch, Rotary_Encoder:RotaryEncoder_Alps_EC11E-Switch_Vertical_H20mm, F.Cu at (150.9, 100.6)
- D1, D10, D11, D12, D2, D3, D4, D5, D6, D7, D8, D9: moved to F.Cu
- moved S10 172.0 mm to (245.8, 41.8), turned to 20 degrees
- moved S9 170.9 mm to (225.4, 41.6), turned to 20 degrees
- moved D10 114.7 mm to (245.4, 52.0), turned to 20 degrees
- moved D9 109.0 mm to (235.7, 41.9), turned to 110 degrees
- moved D1 102.7 mm to (58.6, 48.5), turned to 70 degrees
- moved D11 101.8 mm to (52.1, 66.4), turned to 70 degrees
- moved D8 95.9 mm to (216.9, 46.2), turned to 110 degrees
- moved S8 92.0 mm to (206.7, 45.8), turned to 20 degrees
- moved S7 90.4 mm to (190.4, 56.8), turned to 20 degrees
- moved S6 89.6 mm to (172.5, 63.3), turned to 20 degrees
- moved D2 80.8 mm to (79.0, 48.3), turned to 70 degrees
- moved D12 80.5 mm to (72.5, 66.2), turned to 70 degrees
- moved S11 75.4 mm to (44.5, 59.6), turned to -20 degrees
- moved S12 74.5 mm to (64.8, 59.4), turned to -20 degrees
- moved D7 72.6 mm to (200.7, 57.1), turned to 110 degrees
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Connections:
- D10 pad 1: /Row 2 -> /Row 0
- D11 pad 1: /Row 2 -> /Row 1
- D12 pad 1: /Row 2 -> /Row 1
- D5 pad 1: /Row 1 -> /Row 0
- D6 pad 1: /Row 1 -> /Row 0
- D7 pad 1: /Row 1 -> /Row 0
- D8 pad 1: /Row 1 -> /Row 0
- D9 pad 1: /Row 2 -> /Row 0
- S10 pad 1: /Column 1 -> /Column 9
- S11 pad 1: /Column 2 -> /Column 0
- S12 pad 1: /Column 3 -> /Column 1
- S5 pad 1: /Column 0 -> /Column 4
- S6 pad 1: /Column 1 -> /Column 5
- S7 pad 1: /Column 2 -> /Column 6
- S8 pad 1: /Column 3 -> /Column 7
- S9 pad 1: /Column 0 -> /Column 8
- U1 pad 13: unconnected-(U1-12-Pad13) -> /Encoder A
- U1 pad 14: unconnected-(U1-13-Pad14) -> /Encoder B
- U1 pad 15: unconnected-(U1-14-Pad15) -> /Column 4
- U1 pad 16: unconnected-(U1-15-Pad16) -> /Column 3
- U1 pad 17: unconnected-(U1-26-Pad17) -> /Column 2
- U1 pad 18: unconnected-(U1-27-Pad18) -> /Column 1
- U1 pad 19: unconnected-(U1-28-Pad19) -> /Column 0
- U1 pad 22: unconnected-(U1-GND-Pad22) -> /Encoder C
- U1 pad 4: /Column 0 -> /Row 3
- U1 pad 5: /Column 1 -> /Column 5
- U1 pad 6: /Column 2 -> /Column 6
- U1 pad 7: /Column 3 -> /Column 7
- U1 pad 8: unconnected-(U1-7-Pad8) -> /Column 8
- U1 pad 9: unconnected-(U1-8-Pad9) -> /Column 9
Routing:
- net /Row 3: track 0.00 -> 222.0 mm
- net /Row 2: track 63.5 -> 269.2 mm
- net /Row 1: track 55.9 -> 245.8 mm
- net /Row 0: track 47.0 -> 218.8 mm
- net /Column 9: track 0.00 -> 155.5 mm, vias 0 -> 2
- net /Column 7: track 0.00 -> 141.3 mm, vias 0 -> 2
- net /Column 4: track 0.00 -> 124.9 mm
- net /Column 8: track 0.00 -> 123.8 mm
- net /Column 6: track 0.00 -> 123.6 mm, vias 0 -> 2
- net Net-(D6-A): track 123.1 -> 4.21 mm
- net /Column 5: track 0.00 -> 107.8 mm, vias 0 -> 4
- net /Column 3: track 84.5 -> 186.8 mm, vias 1 -> 2
- net Net-(D5-A): track 112.2 -> 15.4 mm
- net Net-(D1-A): track 94.9 -> 4.21 mm
- net Net-(D9-A): track 85.2 -> 4.21 mm
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Other:
- board size 107.2 x 66.7 mm -> 265 x 144 mm
- board text added: "github.com/sammy-kablammy"
- board text added: "kablamboard"
- board text added: "v1"
- board text removed: "kablampad v0.1"
